File: qfn32_48_lqfn64/breakout_qfn_32_48_lqfn64.kicad_pcb (KiCad board)
At the start: 2 copper layers, 100 x 100 mm, 409 parts, among them J1 TEST_1P, J10 TEST_1P, J100 TEST_1P, J101 TEST_1P, J102 TEST_1P, J103 TEST_1P, J104 TEST_1P, J105 TEST_1P, J106 TEST_1P, J107 TEST_1P, J108 TEST_1P, J109 TEST_1P, J11 TEST_1P, J110 TEST_1P, J111 TEST_1P, J112 TEST_1P, J113 TEST_1P, J114 TEST_1P, J115 TEST_1P, J116 TEST_1P, J117 TEST_1P, J118 TEST_1P, J119 TEST_1P, J12 TEST_1P, J120 TEST_1P, J121 TEST_1P, J122 TEST_1P, J123 TEST_2P, J124 TEST_2P, J125 TEST_2P, J126 TEST_1P, J127 TEST_1P, J128 TEST_1P, J129 TEST_1P, J13 TEST_1P, J130 TEST_1P, J131 TEST_1P, J132 TEST_1P, J133 TEST_1P, J135 TEST_2P, J136 TEST_2P, J137 CONN_02X05, J138 TEST_1P, J139 TEST_1P, J14 TEST_1P, J140 TEST_1P, J141 TEST_1P, J142 TEST_2P, J143 TEST_2P, J144 TEST_2P, J145 TEST_1P, J146 TEST_1P, J147 TEST_1P, J148 TEST_1P, J149 TEST_1P, J15 TEST_1P, J150 TEST_1P, J151 TEST_1P, J152 TEST_1P, J153 TEST_1P, J154 TEST_1P, J155 TEST_1P, J156 TEST_1P, J157 TEST_1P, J158 TEST_1P, J159 TEST_1P, J16 TEST_1P, J160 TEST_1P, J161 TEST_1P, J162 TEST_1P, J163 TEST_1P, J164 TEST_1P, J165 TEST_1P, J166 TEST_1P, J167 TEST_1P, J168 TEST_1P, J169 TEST_1P, J17 TEST_1P, J170 TEST_1P, J171 TEST_1P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

Commit message: errata on name MKL28 instead of mkl26
Other:
- board text added: "MKL26Z FAMILY BREAKOUT BOARD"
Changed lines of the file:
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@@
     (effects (font (size 1.5 1.5) (thickness 0.3)) (justify mirror))
   )
-  (gr_text "MKL28Z FAMILY BREAKOUT BOARD" (at 150 45) (layer B.Mask)
+  (gr_text "MKL26Z FAMILY BREAKOUT BOARD" (at 150 45) (layer B.Mask)
     (effects (font (size 3 3) (thickness 0.5)) (justify mirror))
   )
